File: hardware/v1.0/beltpack_v1_fixed.brd (EAGLE design)
At the start: 100 x 75 mm, 207 parts, among them CN1 Frontpanel, IC1 MEGA32-A, IC10 TS5A9411DCK, IC101 LMR64010, IC11 TS5A9411DCK, IC12 MAX5395LATA+P, IC13 LMV324MZ, IC15 TS5A9411DCK, IC16 LM4880M, IC17 LMV358DGK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

Commit message: added PDF schematics
Routing:
- net 2V5_A: track 100.1 -> 106.5 mm
Changed lines of the file:
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@@
 <wire x1="61.9125" y1="36.305" x2="62.5475" y2="35.67" width="0.254" layer="1"/>
 <contactref element="C61" pad="-"/>
-<wire x1="66.04" y1="68.58" x2="69.5325" y2="67.64" width="0" layer="19" extent="1-1"/>
+<wire x1="69.5325" y1="67.64" x2="69.5325" y2="68.8975" width="0.3" layer="1"/>
+<wire x1="69.5325" y1="68.8975" x2="68.58" y2="69.85" width="0.3" layer="1"/>
+<wire x1="68.58" y1="69.85" x2="64.77" y2="69.85" width="0.3" layer="1"/>
 </signal>
 <signal name="BEEP_AUDIO">
